File: hardware/AMEN_MINI.kicad_pcb (KiCad board)
At the start: 2 copper layers, 114.5 x 168.9 mm, 62 parts, among them J2 Conn_01x04_Pin, J3 Conn_01x14, J4 Conn_01x14, SW1 SW_Push_45deg, SW10 SW_Push_45deg, SW11 SW_Push_45deg, SW12 SW_Push_45deg, SW13 SW_Push_45deg, SW14 SW_Push_45deg, SW15 SW_Push_45deg, SW16 SW_Push_45deg, SW17 SW_Push_45deg, SW18 SW_Push_45deg, SW19 SW_Push_45deg, SW2 SW_Push_45deg, SW20 SW_Push_45deg, SW21 SW_Push_45deg, SW3 SW_Push_45deg, SW4 SW_Push_45deg, SW5 SW_Push_45deg, SW6 SW_Push_45deg, SW7 SW_Push_45deg, SW8 SW_Push_45deg, SW9 SW_Push_45deg, U2 Teensy4.1

Commit message: dont remember what I did here
Parts:
- added G***: LOGO, LOGO, B.Cu at (74.0, 44.8)
Routing:
- net /I2S_MCLK: track 115.2 -> 95.9 mm, vias 3 -> 2
- net /I2S_LRCLK: track 112.5 -> 93.6 mm, vias 3 -> 2
- net /I2S_BCLK: track 97.7 -> 81.6 mm, vias 6 -> 2
- net +3V3: track 216.9 -> 217.8 mm
- net /E5_SW: track 91.9 -> 92.6 mm
- net /ROW0: track 235.4 -> 234.7 mm
- net /+5V_USB: track 85.5 -> 84.9 mm
Other:
- board text added: "+3v3"
- board text added: "GND"
- board text added: "JACK"
- board text added: "MICRO SD"
- board text added: "POWER"
- board text added: "SCL"
- board text added: "SDA"
